Commit message: Add OMY MoveIt config and week 7 IK / planner comparison tools
- omy_moveit_config: SRDF, KDL/LMA/TRAC-IK kinematics, OMPL (RRTConnect),
  joint limits, mock demo / move_group / RViz launch files
- omy_ik_benchmark.py: MoveIt /compute_ik vs our ik_with_restarts on the
  same 300 targets
- omy_moveit_compare.py: our IK vs MoveIt plan vs MoveIt Cartesian, with
  obstacle box and collision re-check
- URDF: link2 collision split into 2 cylinders + box (bounding box overlapped
  link0 when joint2 tilts)
- rviz_mock: camera:=false option, 100 Hz robot_state_publisher

File: src/mobile_manipulator/omy_description/urdf/omy_arm.xacro (robot description, xacro)
@@ -5,5 +5,5 @@
     형상         - ROBOTIS 제공 CAD STL (mm 단위라 scale 0.001)
     질량, COG, 관성 - ROBOTIS 제공 CAD 실측값
-    충돌 형상    - 각 STL 의 바운딩 박스 (직접 계산)
+    충돌 형상    - 각 STL 의 바운딩 박스 (직접 계산), link2 만 원기둥 2 + 박스 1 (아래 설명)
     관절 한계    - 사양서 (joint3 ±150°, 나머지 ±360°), 토크와 속도는 DYNAMIXEL-Y 데이터시트
   0 자세 = 팔이 위로 곧게 선 자세, 플랜지는 link6 의 -y 쪽
@@ -104,9 +104,42 @@
                      xyz="0 ${-omy_shoulder_offset} 0" axis="0 1 0" limit="${2*pi}"
                      effort="${ym080_effort}" velocity="${ym080_velocity}"/>
-    <xacro:omy_link name="link2" mesh="${mesh_dir}/link2.stl" material="omy_light"
-                    box_xyz="0 -0.00155 0.121" box_size="0.087 0.1271 0.329"
-                    mass="3.6795395" com="0.0000114 0.0161842 0.1036063"
-                    ixx="5.1731918e-02" ixy="2.3958819e-06" ixz="5.789396e-05"
-                    iyy="5.0353401e-02" iyz="-4.3825716e-04" izz="4.501436e-03"/>
+    <!-- link2 는 바운딩 박스 대신 STL 모양대로 3 개로 나눔
+         바운딩 박스(0.087 x 0.1271 x 0.329)는 아래 모서리가 joint2 축보다 4.35 cm 아래로 튀어나와
+         joint2 를 기울이면 link0 윗면과 겹침 (READY_POSE 에서도 0.7 mm) → MoveIt 이 충돌로 판정
+         STL 실측 - joint2 하우징 = joint2 축 기준 반지름 43.5 mm, 몸통 폭 77 mm,
+                    joint3 쪽 끝 = joint3 축 기준 반지름 38.5 mm, y 범위는 박스와 같음 -->
+    <link name="link2">
+      <visual>
+        <origin xyz="0 0 0" rpy="0 0 0"/>
+        <geometry>
+          <mesh filename="${mesh_dir}/link2.stl" scale="0.001 0.001 0.001"/>
+        </geometry>
+        <material name="omy_light"/>
+      </visual>
+      <collision>
+        <origin xyz="0 -0.00155 0" rpy="${pi/2} 0 0"/>
+        <geometry>
+          <cylinder radius="0.0435" length="0.1271"/>
+        </geometry>
+      </collision>
+      <collision>
+        <origin xyz="0 -0.00155 ${omy_upper_arm/2}" rpy="0 0 0"/>
+        <geometry>
+          <box size="0.077 0.1271 ${omy_upper_arm}"/>
+        </geometry>
+      </collision>
+      <collision>
+        <origin xyz="0 -0.00155 ${omy_upper_arm}" rpy="${pi/2} 0 0"/>
+        <geometry>
+          <cylinder radius="0.0385" length="0.1271"/>
+        </geometry>
+      </collision>
+      <inertial>
+        <origin xyz="0.0000114 0.0161842 0.1036063" rpy="0 0 0"/>
+        <mass value="3.6795395"/>
+        <inertia ixx="5.1731918e-02" ixy="2.3958819e-06" ixz="5.789396e-05"
+                 iyy="5.0353401e-02" iyz="-4.3825716e-04" izz="4.501436e-03"/>
+      </inertial>
+    </link>
     <!-- 3축 - 팔꿈치 (y), 유일하게 ±150° 로 제한 -->
     <xacro:omy_joint name="joint3" parent="link2" child="link3"
